File: PCB/Designes/I2CFU200/fu200.brd (EAGLE design)
At the start: 100 x 80 mm, 18 parts, among them K1 FINDER-30.22, K2 FINDER-30.22, K3 FINDER-30.22, Q1 BS170, Q2 BS170, Q3 BS170, U1 ATMEGA328P-AU, X1 250-111, X2 250-111

Commit message: Neues Board file
Parts:
- added IC2: LM358N, linear:DIL08
- added MCP4811: (no value), ic-package:DIL08
- added R4: 18k, resistor:0204/7
- added R5: 13k, resistor:0204/7
- added X3: 250-102, con-wago_250:P-250-102
- moved R3 148.8 mm to (-55.9, 95.2), turned to 0 degrees
- moved K3 144.2 mm to (-68.6, 71.1), turned to 0 degrees
- moved Q2 138.6 mm to (-67.3, 88.9)
- moved R2 131.1 mm to (-52.1, 95.2), turned to 0 degrees
- moved D2 130.1 mm to (-59.7, 80.0), turned to 0 degrees
- moved D3 120.2 mm to (-25.4, 90.2), turned to 0 degrees
- moved Q3 118.9 mm to (-22.9, 96.5)
- moved R1 114.3 mm to (-48.3, 95.2), turned to 0 degrees
- moved Q1 113.4 mm to (-54.6, 88.9)
- moved X2 109.1 mm to (-41.9, 25.4), turned to 0 degrees
- moved K2 106.1 mm to (-45.7, 71.1), turned to 0 degrees
- moved D1 98.8 mm to (-39.4, 80.0), turned to 0 degrees
- moved X1 84.7 mm to (-24.1, 25.4), turned to 0 degrees
- moved JP2 83.6 mm to (-41.9, 90.2)
- moved U$1 73.4 mm to (-59.7, 17.8), turned to 0 degrees
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Connections:
- new net N$32: MCP4811.2, U1.32
- new net N$33: IC2.3, MCP4811.8
- new net N$34: MCP4811.3, U1.17
- new net N$35: MCP4811.4, U1.15
- new net N$37: MCP4811.5, U1.1
- new net N$39: IC2.2, R4.1, R5.2
- new net N$40: IC2.1, R4.2, X3.L1
- new net V+: IC2.8
- new net V-: IC2.4
- net N$12: now also U1.2
- net N$13: now also MCP4811.7, R5.1, U1.3, U1.5, X3.L2
- net N$15: now also U1.11
- net N$2: now also MCP4811.1, MCP4811.6
Routing:
- net N$13: track 177.8 -> 0.00 mm
- net N$17: track 77.0 -> 0.00 mm
- net N$23: track 71.6 -> 0.00 mm
- net N$5: track 71.0 -> 0.00 mm
- net N$21: track 66.8 -> 0.00 mm
- net N$14: track 61.4 -> 0.00 mm
- net N$22: track 57.2 -> 0.00 mm
- net N$16: track 50.9 -> 0.00 mm
- net N$20: track 47.8 -> 0.00 mm, vias 1 -> 0
- net N$18: track 40.1 -> 0.00 mm
- net N$6: track 38.3 -> 0.00 mm
- net N$30: track 38.2 -> 0.00 mm
- net N$24: track 37.9 -> 0.00 mm
- net N$19: track 37.2 -> 0.00 mm
- net N$27: track 36.5 -> 0.00 mm
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